Commit message: modified footprint with goetting antennas

File: cob_hardware_config/raw3-1/urdf/raw3-1.urdf.xacro (robot description, xacro)
@@ -41,3 +41,45 @@
       <origin xyz="${gripper_x} ${gripper_y} ${gripper_z}" rpy="${gripper_roll} ${gripper_pitch} ${gripper_yaw}" />
   </xacro:raw_boxgripper>
+  <!-- IMU brick mount on raw3-1 -->
+   <joint name="imu_brick_joint" type="fixed" >
+      <origin xyz="0.495 -0.09250 0.508" rpy="0 0 0" />
+      <parent link="base_link" />
+      <child link="imu_brick_link" />
+    </joint>
+    <link name="imu_brick_link">
+       <inertial>
+            <mass value="0.0001" />
+            <origin xyz="0 0 0" rpy="0 0 0" />
+            <inertia ixx="0.00001" ixy="0" ixz="0" iyy="0.00001" iyz="0" izz="0.00001" />
+       </inertial>
+       <visual>
+               <origin xyz="0 0 -0.02" rpy="0 0 0" />
+            <geometry>
+                   <box size="0.04 0.04 0.02" />
+            </geometry>
+            <material name="IPA/LightGrey" />
+       </visual>
+    </link>
+    <!-- END: IMU brick        mount -->
+    <!-- Softkinetic 'left' mount on raw3-1 -->
+    <joint name="softkinetic_left_joint" type="fixed" >
+      <origin xyz="0.495 0.1125 0.498" rpy="4.3 0.0 ${3*M_PI/2}" />
+      <parent link="base_link" />
+      <child link="softkinetic_left_link" />
+    </joint>
+    <link name="softkinetic_left_link">
+       <inertial>
+            <mass value="0.0001" />
+            <origin xyz="0 0 0" rpy="0 0 0" />
+            <inertia ixx="0.00001" ixy="0" ixz="0" iyy="0.00001" iyz="0" izz="0.00001" />
+       </inertial>
+       <visual>
+               <origin xyz="0 0 0" rpy="0 0 0" />
+            <geometry>
+                   <box size="0.10 0.05 0.03" />
+            </geometry>
+            <material name="IPA/LightGrey" />
+       </visual>
+    </link>
+    <!-- END: Softkinetic 'left' mount -->
   </robot>
